File: Main_Board/PSU.kicad_sch (KiCad schematic)
At the start: 20 parts, among them J3 Baterry input

Commit message: Improve placement/layout
RS485 layout fix, buck-boost, pyro
Parts:
- J3: footprint Connector_PinHeader_2.54mm:PinHeader_1x02_P2.54mm_Vertical -> Connector_JST:JST_PH_B2B-PH-K_1x02_P2.00mm_Vertical
Changed lines of the file:
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@@
 			)
 		)
-		(property "Footprint" "Connector_PinHeader_2.54mm:PinHeader_1x02_P2.54mm_Vertical"
+		(property "Footprint" "Connector_JST:JST_PH_B2B-PH-K_1x02_P2.00mm_Vertical"
 			(at 29.21 80.01 0)
 			(hide yes)

Commit message: Layout/routing/sch
Changed lines of the file:
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@@
 		(dnp no)
 		(property "Reference" "R23"
-			(at 197.866 91.948 90)
+			(at 198.374 92.456 90)
 			(show_name no)
 			(do_not_autoplace no)
@@
 		)
 		(property "Value" "0R"
-			(at 197.358 93.726 90)
+			(at 197.866 94.234 90)
 			(show_name no)
 			(do_not_autoplace no)
@@
 		(dnp no)
 		(property "Reference" "R14"
-			(at 89.154 94.234 0)
+			(at 89.662 93.98 0)
 			(show_name no)
 			(do_not_autoplace no)
@@
 		(dnp no)
 		(property "Reference" "R17"
-			(at 118.872 87.122 90)
+			(at 119.38 87.122 90)
 			(show_name no)
 			(do_not_autoplace no)
@@
 		)
 		(property "Value" "1k"
-			(at 118.872 88.9 90)
+			(at 119.38 88.9 90)
 			(show_name no)
 			(do_not_autoplace no)
@@
 		(dnp no)
 		(property "Reference" "R20"
-			(at 198.374 107.442 0)
+			(at 196.342 108.204 0)
 			(show_name no)
 			(do_not_autoplace no)
@@
 		)
 		(property "Value" "330R"
-			(at 199.644 109.474 0)
+			(at 197.104 110.236 0)
 			(show_name no)
 			(do_not_autoplace no)
@@
 		(dnp no)
 		(property "Reference" "R19"
-			(at 198.374 80.772 0)
+			(at 196.342 81.534 0)
 			(show_name no)
 			(do_not_autoplace no)
@@
 		)
 		(property "Value" "330R"
-			(at 199.644 82.804 0)
+			(at 197.104 83.566 0)
 			(show_name no)
 			(do_not_autoplace no)
@@
 		(dnp no)
 		(property "Reference" "R18"
-			(at 148.844 73.152 0)
+			(at 146.812 73.914 0)
 			(show_name no)
 			(do_not_autoplace no)
@@
 		)
 		(property "Value" "1k"
-			(at 150.114 75.184 0)
+			(at 146.05 75.946 0)
 			(show_name no)
 			(do_not_autoplace no)
@@
 		(dnp no)
 		(property "Reference" "R13"
-			(at 81.788 72.644 90)
+			(at 83.058 73.406 0)
 			(show_name no)
 			(do_not_autoplace no)
@@
 		)
 		(property "Value" "0R"
-			(at 83.566 73.152 90)
-			(show_name no)
-			(do_not_autoplace no)
+			(at 83.566 71.628 0)
+			(show_name no)
+			(do_not_autoplace no)

Commit message: Small fix
Other:
- moved on the sheet: C7, D3, D4, D5, J3, R12, R13, R14, R15, R16, R17, R18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

Commit message: fix shema after review
Parts:
- added R42, R43: 10k, Resistor_SMD:R_0603_1608Metric, symbol Device:R
- R24: value 15k -> 10k
Connections:
- net 3v3_EN: now also R43.1
- net 5V_EN: now also R42.1
- net GND: now also R42.2, R43.2
Other:
- moved on the sheet: D4, D5, R19, R20, R21, R22, R23, R24, R25, R26

Commit message: fix after review -?D7/D8 clamp to 3v3 MB not for 3v3 and other fix
Parts:
- R13: footprint Resistor_SMD:R_0603_1608Metric -> Resistor_SMD:R_0805_2012Metric
Changed lines of the file:
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@@
 			)
 		)
-		(property "Footprint" "Resistor_SMD:R_0603_1608Metric"
+		(property "Footprint" "Resistor_SMD:R_0805_2012Metric"
 			(at 104.648 66.04 90)
 			(hide yes)
