File: Main_Board/Piro_Channels.kicad_sch (KiCad schematic)
At the start: 16 parts, among them J6 Screw_Terminal, J7 Screw_Terminal, Q5 MMBT3904LT1G, Q6 FDN339AN, Q7 MMBT3904LT1G, Q8 FDN339AN

Commit message: Standardise resistor value mark for BOM + pyro footprints
Parts:
- R45, R48, R50, R53: value 10K -> 10k; footprint (none) -> Resistor_SMD:R_0603_1608Metric
- R46, R51: value 100K -> 100k; footprint (none) -> Resistor_SMD:R_0603_1608Metric
- R47, R49, R52, R54: value 1K -> 1k; footprint (none) -> Resistor_SMD:R_0603_1608Metric
Changed lines of the file:
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@@
 			)
 		)
-		(property "Value" "1K"
+		(property "Value" "1k"
 			(at 110.49 93.472 90)
 			(show_name no)
@@
 			)
 		)
-		(property "Footprint" ""
+		(property "Footprint" "Resistor_SMD:R_0603_1608Metric"
 			(at 110.49 99.568 90)
 			(hide yes)
@@
 			)
 		)
-		(property "Value" "10K"
+		(property "Value" "10k"
 			(at 161.29 75.184 90)
 			(show_name no)
@@
 			)
 		)
-		(property "Footprint" ""
+		(property "Footprint" "Resistor_SMD:R_0603_1608Metric"
 			(at 161.29 78.232 90)
 			(hide yes)
@@
 			)
 		)
-		(property "Value" "10K"
+		(property "Value" "10k"
 			(at 105.41 114.3 0)
 			(show_name no)
@@
 			)
 		)
-		(property "Footprint" ""
+		(property "Footprint" "Resistor_SMD:R_0603_1608Metric"
 			(at 110.998 113.03 90)
 			(hide yes)
@@
 			)
 		)
-		(property "Value" "100K"
+		(property "Value" "100k"
 			(at 91.44 93.472 90)
 			(show_name no)
@@
 			)
 		)
-		(property "Footprint" ""
+		(property "Footprint" "Resistor_SMD:R_0603_1608Metric"
 			(at 91.44 99.568 90)
 			(hide yes)
@@
 			)
 		)
-		(property "Value" "1K"
+		(property "Value" "1k"
 			(at 187.96 102.362 90)
 			(show_name no)
@@
 			)
 		)
-		(property "Footprint" ""
+		(property "Footprint" "Resistor_SMD:R_0603_1608Metric"
 			(at 187.96 108.458 90)
 			(hide yes)
@@
 			)
 		)
-		(property "Value" "10K"
+		(property "Value" "10k"
 			(at 74.93 75.184 90)
 			(show_name no)
@@
 			)
 		)
-		(property "Footprint" ""
+		(property "Footprint" "Resistor_SMD:R_0603_1608Metric"
 			(at 74.93 78.232 90)
 			(hide yes)
@@
 			)
 		)
-		(property "Value" "10K"
+		(property "Value" "10k"
 			(at 191.77 114.3 0)
 			(show_name no)
@@
 			)
 		)
-		(property "Footprint" ""
+		(property "Footprint" "Resistor_SMD:R_0603_1608Metric"
 			(at 197.358 113.03 90)
 			(hide yes)
@@
 			)
 		)
-		(property "Value" "1K"
+		(property "Value" "1k"
 			(at 196.85 93.472 90)
 			(show_name no)
@@
 			)
 		)
-		(property "Footprint" ""
+		(property "Footprint" "Resistor_SMD:R_0603_1608Metric"
 			(at 196.85 99.568 90)
 			(hide yes)
@@
 			)
 		)
-		(property "Value" "100K"
+		(property "Value" "100k"
 			(at 177.8 93.472 90)
 			(show_name no)
@@
 			)
 		)
-		(property "Footprint" ""
+		(property "Footprint" "Resistor_SMD:R_0603_1608Metric"
 			(at 177.8 99.568 90)
 			(hide yes)
@@
 			)
 		)
-		(property "Value" "1K"
+		(property "Value" "1k"
 			(at 101.6 102.362 90)
 			(show_name no)
@@
 			)
 		)
-		(property "Footprint" ""
+		(property "Footprint" "Resistor_SMD:R_0603_1608Metric"
 			(at 101.6 108.458 90)
 			(hide yes)

Commit message: Pyro layout + schematic fix
Parts:
- removed J6, J7: Screw_Terminal, symbol Connector:Screw_Terminal_01x02
- removed Q5, Q7: MMBT3904LT1G, Package_TO_SOT_SMD:SOT-23, symbol Simulation_SPICE:NPN
- removed Q6, Q8: FDN339AN, Package_TO_SOT_SMD:SOT-23, symbol Device:Q_NMOS_GDS
- removed R45, R48, R50, R53: 10k, Resistor_SMD:R_0603_1608Metric, symbol Device:R
- removed R46, R51: 100k, Resistor_SMD:R_0603_1608Metric, symbol Device:R
- removed R47, R49, R52, R54: 1k, Resistor_SMD:R_0603_1608Metric, symbol Device:R
Other:
- added sheet Pyro_Channel1 (PyroChannel1.kicad_sch)
- added sheet Pyro_Channel2 (PyroChannel1.kicad_sch)
