File: Main_Board/PyroChannel1.kicad_sch (KiCad schematic)
At the start: 8 parts, among them J7 Screw_Terminal, Q7 MMBT3904LT1G, Q8 FDN339AN

Commit message: Layout
Parts:
- added C42: 470uF, Capacitor_THT:CP_Radial_D4.0mm_P2.00mm, symbol Device:C_Polarized
- J7: value Screw_Terminal -> Terminal
Connections:
- net GND: now also C42.2
- net VBUS: now also C42.1

Commit message: New footprints + layout
Parts:
- J7: footprint (none) -> SamacSys_Parts:SHDR2W80P0X381_1X2_841X700X920P
Changed lines of the file:
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@@
 			)
 		)
-		(property "Footprint" ""
+		(property "Footprint" "SamacSys_Parts:SHDR2W80P0X381_1X2_841X700X920P"
 			(at 166.37 93.98 0)
 			(hide yes)

Commit message: layout update
Parts:
- C42: footprint Capacitor_THT:CP_Radial_D4.0mm_P2.00mm -> Capacitor_SMD:CP_Elec_8x10
Changed lines of the file:
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@@
 			)
 		)
-		(property "Footprint" "Capacitor_THT:CP_Radial_D4.0mm_P2.00mm"
+		(property "Footprint" "Capacitor_SMD:CP_Elec_8x10"
 			(at 185.1152 120.65 0)
 			(hide yes)

Commit message: Schematic cleanup, ALED footprint + 3D + sch
+ layout and routing
Other:
- moved on the sheet: C42, J7, Q7, Q8, R50, R51, R52, R53, R54

Commit message: nettie add /gnd split
Connections:
- net GND: no longer C42.2, Q8.2 (S), R53.1
- new net GNDPWR: C42.2, Q8.2 (S), R53.1
Changed lines of the file:
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@@
 	)
 	(symbol
-		(lib_id "power:GND")
-		(at 119.38 125.73 0)
+		(lib_id "power:GNDPWR")
+		(at 182.88 125.73 0)
 		(unit 1)
 		(body_style 1)
@@
 		(dnp no)
 		(fields_autoplaced yes)
-		(property "Reference" "#PWR0106"
-			(at 119.38 132.08 0)
-			(hide yes)
-			(show_name no)
-			(do_not_autoplace no)
-			(effects
-				(font
-					(size 1.27 1.27)
-				)
-			)
-		)
-		(property "Value" "GND"
-			(at 119.38 130.81 0)
-			(hide yes)
+		(property "Reference" "#PWR083"
+			(at 182.88 130.81 0)
+			(hide yes)
+			(show_name no)
+			(do_not_autoplace no)
+			(effects
+				(font
+					(size 1.27 1.27)
+				)
+			)
+		)
+		(property "Value" "GNDPWR"
+			(at 182.753 129.54 0)
 			(show_name no)
 			(do_not_autoplace no)
@@
 		)
 		(property "Footprint" ""
-			(at 119.38 125.73 0)
+			(at 182.88 127 0)
 			(hide yes)
 			(show_name no)
@@
 		)
 		(property "Datasheet" ""
-			(at 119.38 125.73 0)
-			(hide yes)
-			(show_name no)
-			(do_not_autoplace no)
-			(effects
-				(font
-					(size 1.27 1.27)
-				)
-			)
-		)
-		(property "Description" ""
-			(at 119.38 125.73 0)
-			(hide yes)
-			(show_name no)
-			(do_not_autoplace no)
-			(effects
-				(font
-					(size 1.27 1.27)
-				)
-			)
-		)
-		(pin "1"
-		)
-		(instances
-			(project "Main_Board"
-				(path "/7481738f-7c20-40bb-99b0-6ccd4168db33/a9efd6b0-2353-4b74-9b2e-55e0801cf9fc/8a13c8a5-8054-4bf0-abea-4a33e90adbcf"
-					(reference "#PWR0110")
-					(unit 1)
-				)
-				(path "/7481738f-7c20-40bb-99b0-6ccd4168db33/a9efd6b0-2353-4b74-9b2e-55e0801cf9fc/cd6734be-dc35-4322-bfb0-ed11c8242097"
-					(reference "#PWR0106")
+			(at 182.88 127 0)
+			(hide yes)
+			(show_name no)
+			(do_not_autoplace no)
+			(effects
+				(font
+					(size 1.27 1.27)
+				)
+			)
+		)
+		(property "Description" "Power symbol creates a global label with name \"GNDPWR\" , global ground"
+			(at 182.88 125.73 0)
+			(hide yes)
+			(show_name no)
+			(do_not_autoplace no)
+			(effects
+				(font
+					(size 1.27 1.27)
+				)
+			)
+		)
+		(pin "1"
+		)
+		(instances
+			(project "Main_Board"
+				(path "/7481738f-7c20-40bb-99b0-6ccd4168db33/a9efd6b0-2353-4b74-9b2e-55e0801cf9fc/8a13c8a5-8054-4bf0-abea-4a33e90adbcf"
+					(reference "#PWR084")
+					(unit 1)
+				)
+				(path "/7481738f-7c20-40bb-99b0-6ccd4168db33/a9efd6b0-2353-4b74-9b2e-55e0801cf9fc/cd6734be-dc35-4322-bfb0-ed11c8242097"
+					(reference "#PWR083")
 					(unit 1)
 				)
@@
 				(path "/7481738f-7c20-40bb-99b0-6ccd4168db33/a9efd6b0-2353-4b74-9b2e-55e0801cf9fc/cd6734be-dc35-4322-bfb0-ed11c8242097"
 					(reference "R54")
-					(unit 1)
-				)
-			)
-		)
-	)
-	(symbol
-		(lib_id "power:GND")
-		(at 154.94 125.73 0)
-		(unit 1)
-		(body_style 1)
-		(exclude_from_sim no)
-		(in_bom yes)
-		(on_board yes)
-		(in_pos_files yes)
-		(dnp no)
-		(fields_autoplaced yes)
-		(property "Reference" "#PWR0107"
-			(at 154.94 132.08 0)
-			(hide yes)
-			(show_name no)
-			(do_not_autoplace no)
-			(effects
-				(font
-					(size 1.27 1.27)
-				)
-			)
-		)
-		(property "Value" "GND"
-			(at 154.94 130.81 0)
-			(hide yes)
-			(show_name no)
-			(do_not_autoplace no)
-			(effects
-				(font
-					(size 1.27 1.27)
-				)
-			)
-		)
-		(property "Footprint" ""
-			(at 154.94 125.73 0)
-			(hide yes)
-			(show_name no)
-			(do_not_autoplace no)
-			(effects
-				(font
-					(size 1.27 1.27)
-				)
-			)
-		)
-		(property "Datasheet" ""
-			(at 154.94 125.73 0)
-			(hide yes)
-			(show_name no)
-			(do_not_autoplace no)
-			(effects
-				(font
-					(size 1.27 1.27)
-				)
-			)
-		)
-		(property "Description" ""
-			(at 154.94 125.73 0)
-			(hide yes)
-			(show_name no)
-			(do_not_autoplace no)
-			(effects
-				(font
-					(size 1.27 1.27)
-				)
-			)
-		)
-		(pin "1"
-		)
-		(instances
-			(project "Main_Board"
-				(path "/7481738f-7c20-40bb-99b0-6ccd4168db33/a9efd6b0-2353-4b74-9b2e-55e0801cf9fc/8a13c8a5-8054-4bf0-abea-4a33e90adbcf"
-					(reference "#PWR0111")
-					(unit 1)
-				)
-				(path "/7481738f-7c20-40bb-99b0-6ccd4168db33/a9efd6b0-2353-4b74-9b2e-55e0801cf9fc/cd6734be-dc35-4322-bfb0-ed11c8242097"
-					(reference "#PWR0107")
 					(unit 1)
 				)
@@
 	)
 	(symbol
-		(lib_id "power:GND")
-		(at 182.88 125.73 0)
-		(unit 1)
-		(body_style 1)
-		(exclude_from_sim no)
-		(in_bom yes)
-		(on_board yes)
-		(in_pos_files yes)
-		(dnp no)
-		(fields_autoplaced yes)
-		(property "Reference" "#PWR0115"
-			(at 182.88 132.08 0)
-			(hide yes)
-			(show_name no)
-			(do_not_autoplace no)
-			(effects
-				(font
-					(size 1.27 1.27)
-				)
-			)
-		)
-		(property "Value" "GND"
-			(at 182.88 130.81 0)
-			(hide yes)
-			(show_name no)
-			(do_not_autoplace no)
-			(effects
-				(font
-					(size 1.27 1.27)
-				)
-			)
-		)
-		(property "Footprint" ""
-			(at 182.88 125.73 0)
-			(hide yes)
-			(show_name no)
-			(do_not_autoplace no)
-			(effects
-				(font
-					(size 1.27 1.27)
-				)
-			)
-		)
-		(property "Datasheet" ""
-			(at 182.88 125.73 0)
-			(hide yes)
-			(show_name no)
-			(do_not_autoplace no)
-			(effects
-				(font
-					(size 1.27 1.27)
-				)
-			)
-		)
-		(property "Description" ""
-			(at 182.88 125.73 0)
-			(hide yes)
-			(show_name no)
-			(do_not_autoplace no)
-			(effects
-				(font
-					(size 1.27 1.27)
-				)
-			)
-		)
-		(pin "1"
-		)
-		(instances
-			(project "Main_Board"
-				(path "/7481738f-7c20-40bb-99b0-6ccd4168db33/a9efd6b0-2353-4b74-9b2e-55e0801cf9fc/8a13c8a5-8054-4bf0-abea-4a33e90adbcf"
-					(reference "#PWR0116")
-					(unit 1)
-				)
-				(path "/7481738f-7c20-40bb-99b0-6ccd4168db33/a9efd6b0-2353-4b74-9b2e-55e0801cf9fc/cd6734be-dc35-4322-bfb0-ed11c8242097"
-					(reference "#PWR0115")
-					(unit 1)
-				)
-			)
-		)
-	)
-	(symbol
 		(lib_id "Device:R")
 		(at 129.54 101.6 90)
@@
 					(unit 1)
 				)
+			)
+		)
+	)
+	(symbol
+		(lib_id "power:GND")
+		(at 119.38 125.73 0)
+		(unit 1)
+		(body_style 1)
+		(exclude_from_sim no)
+		(in_bom yes)
+		(on_board yes)
+		(in_pos_files yes)
+		(dnp no)
+		(fields_autoplaced yes)
+		(property "Reference" "#PWR067"
+			(at 119.38 132.08 0)
+			(hide yes)
+			(show_name no)
+			(do_not_autoplace no)
+			(effects
+				(font
+					(size 1.27 1.27)
+				)
+			)
+		)
+		(property "Value" "GND"
+			(at 119.38 130.81 0)
+			(show_name no)
+			(do_not_autoplace no)
+			(effects
+				(font
+					(size 1.27 1.27)
+				)
+			)
+		)
+		(property "Footprint" ""
+			(at 119.38 125.73 0)
+			(hide yes)
+			(show_name no)
+			(do_not_autoplace no)
+			(effects
+				(font
+					(size 1.27 1.27)
+				)
+			)
+		)
+		(property "Datasheet" ""
+			(at 119.38 125.73 0)
+			(hide yes)
+			(show_name no)
+			(do_not_autoplace no)
+			(effects
+				(font
+					(size 1.27 1.27)
+				)
+			)
+		)
+		(property "Description" "Power symbol creates a global label with name \"GND\" , ground"
+			(at 119.38 125.73 0)
+			(hide yes)
+			(show_name no)
+			(do_not_autoplace no)
+			(effects
+				(font
+					(size 1.27 1.27)
+				)
+			)
+		)
+		(pin "1"
+		)
+		(instances
+			(project "Main_Board"
+				(path "/7481738f-7c20-40bb-99b0-6ccd4168db33/a9efd6b0-2353-4b74-9b2e-55e0801cf9fc/8a13c8a5-8054-4bf0-abea-4a33e90adbcf"
+					(reference "#PWR068")
+					(unit 1)
+				)
+				(path "/7481738f-7c20-40bb-99b0-6ccd4168db33/a9efd6b0-2353-4b74-9b2e-55e0801cf9fc/cd6734be-dc35-4322-bfb0-ed11c8242097"
+					(reference "#PWR067")
+					(unit 1)
+				)
+			)
+		)
+	)
+	(symbol
+		(lib_id "power:GNDPWR")
+		(at 154.94 125.73 0)
+		(unit 1)
+		(body_style 1)
+		(exclude_from_sim no)
+		(in_bom yes)
+		(on_board yes)
+		(in_pos_files yes)
+		(dnp no)
+		(fields_autoplaced yes)
+		(property "Reference" "#PWR071"
+			(at 154.94 130.81 0)
+			(hide yes)
+			(show_name no)
+			(do_not_autoplace no)
+			(effects
+				(font
+					(size 1.27 1.27)
+				)
+			)
+		)
+		(property "Value" "GNDPWR"
+			(at 154.813 129.54 0)
+			(show_name no)
+			(do_not_autoplace no)
+			(effects
+				(font
+					(size 1.27 1.27)
+				)
+			)
+		)
+		(property "Footprint" ""
+			(at 154.94 127 0)
+			(hide yes)
+			(show_name no)
+			(do_not_autoplace no)
+			(effects
+				(font
+					(size 1.27 1.27)
+				)
+			)
+		)
+		(property "Datasheet" ""
+			(at 154.94 127 0)
+			(hide yes)
+			(show_name no)
+			(do_not_autoplace no)
+			(effects
+				(font
+					(size 1.27 1.27)
+				)
+			)
+		)
+		(property "Description" "Power symbol creates a global label with name \"GNDPWR\" , global ground"
+			(at 154.94 125.73 0)
+			(hide yes)
+			(show_name no)
+			(do_not_autoplace no)
+			(effects
+				(font
+					(size 1.27 1.27)
+				)
+			)
+		)
+		(pin "1"
+		)
+		(instances
+			(project "Main_Board"
+				(path "/7481738f-7c20-40bb-99b0-6ccd4168db33/a9efd6b0-2353-4b74-9b2e-55e0801cf9fc/8a13c8a5-8054-4bf0-abea-4a33e90adbcf"
+					(reference "#PWR072")
+					(unit 1)
+				)
+				(path "/7481738f-7c20-40bb-99b0-6ccd4168db33/a9efd6b0-2353-4b74-9b2e-55e0801cf9fc/cd6734be-dc35-4322-bfb0-ed11c8242097"
+					(reference "#PWR071")
+					(unit 1)
+				)

Commit message: Pyro fix + silk
Parts:
- R54: value 1k -> 47k
Changed lines of the file:
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@@
 			)
 		)
-		(property "Value" "1k"
+		(property "Value" "47k"
 			(at 151.13 97.282 90)
 			(show_name no)
