File: Main_Board/UART_RS485_Transciever.kicad_sch (KiCad schematic)
At the start: 10 parts, among them U6 THVD1450DR

Commit message: Aesthetics/cleanup
Connections:
- net ESP_UART_DIR renamed TRANSCIEVER_UART_DIR
- net ESP_UART_RX renamed TRANSCIEVER_UART_RX
- net ESP_UART_TX renamed TRANSCIEVER_UART_TX
Other:
- note added: "Add DIP switches on modules to toggle the 120 ohm termination resistor on the bus"
Changed lines of the file:
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@@
 	(generator_version "10.0")
 	(paper "A4")
+	(text "Add DIP switches on modules to toggle the \n120 ohm termination resistor on the bus"
+		(exclude_from_sim no)
+		(at 188.976 110.744 0)
+		(effects
+			(font
+				(size 1.27 1.27)
+			)
+			(justify left)
+		)
+	)
 	(junction
 		(at 133.35 118.11)
@@
 		)
 	)
-	(hierarchical_label "ESP_UART_RX"
-		(shape input)
+	(hierarchical_label "TRANSCIEVER_UART_RX"
+		(shape output)
 		(at 93.98 95.25 180)
 		(effects
@@
 		)
 	)
-	(hierarchical_label "ESP_UART_DIR"
+	(hierarchical_label "TRANSCIEVER_UART_DIR"
 		(shape input)
 		(at 93.98 100.33 180)
@@
 		)
 	)
-	(hierarchical_label "ESP_UART_TX"
-		(shape output)
+	(hierarchical_label "TRANSCIEVER_UART_TX"
+		(shape input)
 		(at 93.98 105.41 180)
 		(effects

Commit message: add external obrds interfaces
Todo pyro chanells
Changed lines of the file:
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@@
 	(text "Add DIP switches on modules to toggle the \n120 ohm termination resistor on the bus"
 		(exclude_from_sim no)
-		(at 188.976 110.744 0)
+		(at 171.958 118.11 0)
 		(effects
 			(font

Commit message: Add buzzer, Add LED, ADD R&D jumper
Parts:
- renumbered C32 to C39, C30 to C40, C31 to C41, D9 to D12, R26 to R33, R25 to R34, R28 to R35, R27 to R36, R29 to R37, U6 to U7
Changed lines of the file:
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@@
 		(in_pos_files yes)
 		(dnp no)
-		(property "Reference" "D9"
+		(property "Reference" "D12"
 			(at 181.102 80.264 90)
 			(show_name no)
@@
 			(project "Main_Board"
 				(path "/7481738f-7c20-40bb-99b0-6ccd4168db33/f339aa79-d1b1-4b60-b951-815db04e9281/9134e59b-c18f-4136-baaa-a4c593015be7"
-					(reference "D9")
+					(reference "D12")
 					(unit 1)
 				)
@@
 		(in_pos_files yes)
 		(dnp no)
-		(property "Reference" "R25"
+		(property "Reference" "R34"
 			(at 129.794 110.49 0)
 			(show_name no)
@@
 			(project "Main_Board"
 				(path "/7481738f-7c20-40bb-99b0-6ccd4168db33/f339aa79-d1b1-4b60-b951-815db04e9281/9134e59b-c18f-4136-baaa-a4c593015be7"
-					(reference "R25")
+					(reference "R34")
 					(unit 1)
 				)
@@
 		(in_pos_files yes)
 		(dnp no)
-		(property "Reference" "#PWR060"
+		(property "Reference" "#PWR089"
 			(at 133.35 128.27 0)
 			(hide yes)
@@
 			(project "Main_Board"
 				(path "/7481738f-7c20-40bb-99b0-6ccd4168db33/f339aa79-d1b1-4b60-b951-815db04e9281/9134e59b-c18f-4136-baaa-a4c593015be7"
-					(reference "#PWR060")
+					(reference "#PWR089")
 					(unit 1)
 				)
@@
 		(in_pos_files yes)
 		(dnp no)
-		(property "Reference" "#PWR062"
+		(property "Reference" "#PWR090"
 			(at 135.89 95.25 0)
 			(hide yes)
@@
 			(project "Main_Board"
 				(path "/7481738f-7c20-40bb-99b0-6ccd4168db33/f339aa79-d1b1-4b60-b951-815db04e9281/9134e59b-c18f-4136-baaa-a4c593015be7"
-					(reference "#PWR062")
+					(reference "#PWR090")
 					(unit 1)
 				)
@@
 		(in_pos_files yes)
 		(dnp no)
-		(property "Reference" "C30"
+		(property "Reference" "C40"
 			(at 125.73 82.55 0)
 			(show_name no)
@@
 			(project "Main_Board"
 				(path "/7481738f-7c20-40bb-99b0-6ccd4168db33/f339aa79-d1b1-4b60-b951-815db04e9281/9134e59b-c18f-4136-baaa-a4c593015be7"
-					(reference "C30")
+					(reference "C40")
 					(unit 1)
 				)
@@
 		(in_pos_files yes)
 		(dnp no)
-		(property "Reference" "R27"
+		(property "Reference" "R36"
 			(at 167.386 102.87 90)
 			(show_name no)
@@
 			(project "Main_Board"
 				(path "/7481738f-7c20-40bb-99b0-6ccd4168db33/f339aa79-d1b1-4b60-b951-815db04e9281/9134e59b-c18f-4136-baaa-a4c593015be7"
-					(reference "R27")
+					(reference "R36")
 					(unit 1)
 				)
@@
 		(in_pos_files yes)
 		(dnp no)
-		(property "Reference" "C32"
+		(property "Reference" "C39"
 			(at 113.03 82.55 0)
 			(show_name no)
@@
 			(project "Main_Board"
 				(path "/7481738f-7c20-40bb-99b0-6ccd4168db33/f339aa79-d1b1-4b60-b951-815db04e9281/9134e59b-c18f-4136-baaa-a4c593015be7"
-					(reference "C32")
+					(reference "C39")
 					(unit 1)
 				)
@@
 		(in_pos_files yes)
 		(dnp no)
-		(property "Reference" "#PWR063"
+		(property "Reference" "#PWR092"
 			(at 181.61 114.3 0)
 			(hide yes)
@@
 			(project "Main_Board"
 				(path "/7481738f-7c20-40bb-99b0-6ccd4168db33/f339aa79-d1b1-4b60-b951-815db04e9281/9134e59b-c18f-4136-baaa-a4c593015be7"
-					(reference "#PWR063")
+					(reference "#PWR092")
 					(unit 1)
 				)
@@
 		(in_pos_files yes)
 		(dnp no)
-		(property "Reference" "U6"
+		(property "Reference" "U7"
 			(at 151.13 115.57 0)
 			(show_name no)
@@
 			(project "Main_Board"
 				(path "/7481738f-7c20-40bb-99b0-6ccd4168db33/f339aa79-d1b1-4b60-b951-815db04e9281/9134e59b-c18f-4136-baaa-a4c593015be7"
-					(reference "U6")
+					(reference "U7")
 					(unit 1)
 				)
@@
 		(in_pos_files yes)
 		(dnp no)
-		(property "Reference" "R28"
+		(property "Reference" "R35"
 			(at 167.894 87.63 90)
 			(show_name no)
@@
 			(project "Main_Board"
 				(path "/7481738f-7c20-40bb-99b0-6ccd4168db33/f339aa79-d1b1-4b60-b951-815db04e9281/9134e59b-c18f-4136-baaa-a4c593015be7"
-					(reference "R28")
+					(reference "R35")
 					(unit 1)
 				)
@@
 		(in_pos_files yes)
 		(dnp no)
-		(property "Reference" "#PWR061"
+		(property "Reference" "#PWR088"
 			(at 123.19 95.25 0)
 			(hide yes)
@@
 			(project "Main_Board"
 				(path "/7481738f-7c20-40bb-99b0-6ccd4168db33/f339aa79-d1b1-4b60-b951-815db04e9281/9134e59b-c18f-4136-baaa-a4c593015be7"
-					(reference "#PWR061")
+					(reference "#PWR088")
 					(unit 1)
 				)
@@
 		(dnp no)
 		(fields_autoplaced yes)
-		(property "Reference" "#PWR064"
+		(property "Reference" "#PWR091"
 			(at 149.86 80.01 0)
 			(hide yes)
@@
 			(project "Main_Board"
 				(path "/7481738f-7c20-40bb-99b0-6ccd4168db33/f339aa79-d1b1-4b60-b951-815db04e9281/9134e59b-c18f-4136-baaa-a4c593015be7"
-					(reference "#PWR064")
+					(reference "#PWR091")
 					(unit 1)
 				)
@@
 		(in_pos_files yes)
 		(dnp no)
-		(property "Reference" "R29"
+		(property "Reference" "R37"
 			(at 194.564 96.52 0)
 			(show_name no)
@@
 			(project "Main_Board"
 				(path "/7481738f-7c20-40bb-99b0-6ccd4168db33/f339aa79-d1b1-4b60-b951-815db04e9281/9134e59b-c18f-4136-baaa-a4c593015be7"
-					(reference "R29")
+					(reference "R37")
 					(unit 1)
 				)
@@
 		(in_pos_files yes)
 		(dnp no)
-		(property "Reference" "R26"
+		(property "Reference" "R33"
 			(at 95.504 85.09 0)
 			(show_name no)
@@
 			(project "Main_Board"
 				(path "/7481738f-7c20-40bb-99b0-6ccd4168db33/f339aa79-d1b1-4b60-b951-815db04e9281/9134e59b-c18f-4136-baaa-a4c593015be7"
-					(reference "R26")
+					(reference "R33")
 					(unit 1)
 				)
@@
 		(in_pos_files yes)
 		(dnp no)
-		(property "Reference" "C31"
+		(property "Reference" "C41"
 			(at 138.43 82.55 0)
 			(show_name no)
@@
 			(project "Main_Board"
 				(path "/7481738f-7c20-40bb-99b0-6ccd4168db33/f339aa79-d1b1-4b60-b951-815db04e9281/9134e59b-c18f-4136-baaa-a4c593015be7"
-					(reference "C31")
+					(reference "C41")
 					(unit 1)
 				)
@@
 		(in_pos_files yes)
 		(dnp no)
-		(property "Reference" "#PWR065"
+		(property "Reference" "#PWR087"
 			(at 110.49 95.25 0)
 			(hide yes)
@@
 			(project "Main_Board"
 				(path "/7481738f-7c20-40bb-99b0-6ccd4168db33/f339aa79-d1b1-4b60-b951-815db04e9281/9134e59b-c18f-4136-baaa-a4c593015be7"
-					(reference "#PWR065")
-					(unit 1)
-				)
+					(reference "#PWR087")
+					(unit 1)
+				)

Commit message: ADD footprints
Parts:
- C39, C40, C41: footprint (none) -> Capacitor_SMD:C_0603_1608Metric
- R33, R34, R35, R36, R37: footprint (none) -> Resistor_SMD:R_0603_1608Metric
Changed lines of the file:
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@@
 			)
 		)
-		(property "Footprint" ""
+		(property "Footprint" "Resistor_SMD:R_0603_1608Metric"
 			(at 135.128 111.76 90)
 			(hide yes)
@@
 			)
 		)
-		(property "Footprint" ""
+		(property "Footprint" "Capacitor_SMD:C_0603_1608Metric"
 			(at 124.1552 87.63 0)
 			(hide yes)
@@
 			)
 		)
-		(property "Footprint" ""
+		(property "Footprint" "Resistor_SMD:R_0603_1608Metric"
 			(at 167.64 96.012 90)
 			(hide yes)
@@
 			)
 		)
-		(property "Footprint" ""
+		(property "Footprint" "Capacitor_SMD:C_0603_1608Metric"
 			(at 111.4552 87.63 0)
 			(hide yes)
@@
 			)
 		)
-		(property "Footprint" ""
+		(property "Footprint" "Resistor_SMD:R_0603_1608Metric"
 			(at 167.64 94.488 90)
 			(hide yes)
@@
 			)
 		)
-		(property "Footprint" ""
+		(property "Footprint" "Resistor_SMD:R_0603_1608Metric"
 			(at 199.898 95.25 90)
 			(hide yes)
@@
 			)
 		)
-		(property "Footprint" ""
+		(property "Footprint" "Resistor_SMD:R_0603_1608Metric"
 			(at 100.838 86.36 90)
 			(hide yes)
@@
 			)
 		)
-		(property "Footprint" ""
+		(property "Footprint" "Capacitor_SMD:C_0603_1608Metric"
 			(at 136.8552 87.63 0)
 			(hide yes)

Commit message: Add pyro channels x2
Parts:
- renumbered R33 to R35, R34 to R36, R35 to R37, R36 to R38, R37 to R39
Changed lines of the file:
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@@
 		(in_pos_files yes)
 		(dnp no)
-		(property "Reference" "R34"
+		(property "Reference" "R36"
 			(at 129.794 110.49 0)
 			(show_name no)
@@
 			(project "Main_Board"
 				(path "/7481738f-7c20-40bb-99b0-6ccd4168db33/f339aa79-d1b1-4b60-b951-815db04e9281/9134e59b-c18f-4136-baaa-a4c593015be7"
-					(reference "R34")
+					(reference "R36")
 					(unit 1)
 				)
@@
 		(in_pos_files yes)
 		(dnp no)
-		(property "Reference" "#PWR089"
+		(property "Reference" "#PWR093"
 			(at 133.35 128.27 0)
 			(hide yes)
@@
 			(project "Main_Board"
 				(path "/7481738f-7c20-40bb-99b0-6ccd4168db33/f339aa79-d1b1-4b60-b951-815db04e9281/9134e59b-c18f-4136-baaa-a4c593015be7"
-					(reference "#PWR089")
+					(reference "#PWR093")
 					(unit 1)
 				)
@@
 		(in_pos_files yes)
 		(dnp no)
-		(property "Reference" "#PWR090"
+		(property "Reference" "#PWR094"
 			(at 135.89 95.25 0)
 			(hide yes)
@@
 			(project "Main_Board"
 				(path "/7481738f-7c20-40bb-99b0-6ccd4168db33/f339aa79-d1b1-4b60-b951-815db04e9281/9134e59b-c18f-4136-baaa-a4c593015be7"
-					(reference "#PWR090")
+					(reference "#PWR094")
 					(unit 1)
 				)
@@
 		(in_pos_files yes)
 		(dnp no)
-		(property "Reference" "R36"
+		(property "Reference" "R38"
 			(at 167.386 102.87 90)
 			(show_name no)
@@
 			(project "Main_Board"
 				(path "/7481738f-7c20-40bb-99b0-6ccd4168db33/f339aa79-d1b1-4b60-b951-815db04e9281/9134e59b-c18f-4136-baaa-a4c593015be7"
-					(reference "R36")
+					(reference "R38")
 					(unit 1)
 				)
@@
 		(in_pos_files yes)
 		(dnp no)
-		(property "Reference" "#PWR092"
+		(property "Reference" "#PWR096"
 			(at 181.61 114.3 0)
 			(hide yes)
@@
 			(project "Main_Board"
 				(path "/7481738f-7c20-40bb-99b0-6ccd4168db33/f339aa79-d1b1-4b60-b951-815db04e9281/9134e59b-c18f-4136-baaa-a4c593015be7"
-					(reference "#PWR092")
+					(reference "#PWR096")
 					(unit 1)
 				)
@@
 		(in_pos_files yes)
 		(dnp no)
-		(property "Reference" "R35"
+		(property "Reference" "R37"
 			(at 167.894 87.63 90)
 			(show_name no)
@@
 			(project "Main_Board"
 				(path "/7481738f-7c20-40bb-99b0-6ccd4168db33/f339aa79-d1b1-4b60-b951-815db04e9281/9134e59b-c18f-4136-baaa-a4c593015be7"
-					(reference "R35")
+					(reference "R37")
 					(unit 1)
 				)
@@
 		(in_pos_files yes)
 		(dnp no)
-		(property "Reference" "#PWR088"
+		(property "Reference" "#PWR092"
 			(at 123.19 95.25 0)
 			(hide yes)
@@
 			(project "Main_Board"
 				(path "/7481738f-7c20-40bb-99b0-6ccd4168db33/f339aa79-d1b1-4b60-b951-815db04e9281/9134e59b-c18f-4136-baaa-a4c593015be7"
-					(reference "#PWR088")
+					(reference "#PWR092")
 					(unit 1)
 				)
@@
 		(dnp no)
 		(fields_autoplaced yes)
-		(property "Reference" "#PWR091"
+		(property "Reference" "#PWR095"
 			(at 149.86 80.01 0)
 			(hide yes)
@@
 			(project "Main_Board"
 				(path "/7481738f-7c20-40bb-99b0-6ccd4168db33/f339aa79-d1b1-4b60-b951-815db04e9281/9134e59b-c18f-4136-baaa-a4c593015be7"
-					(reference "#PWR091")
+					(reference "#PWR095")
 					(unit 1)
 				)
@@
 		(in_pos_files yes)
 		(dnp no)
-		(property "Reference" "R37"
+		(property "Reference" "R39"
 			(at 194.564 96.52 0)
 			(show_name no)
@@
 			(project "Main_Board"
 				(path "/7481738f-7c20-40bb-99b0-6ccd4168db33/f339aa79-d1b1-4b60-b951-815db04e9281/9134e59b-c18f-4136-baaa-a4c593015be7"
-					(reference "R37")
+					(reference "R39")
 					(unit 1)
 				)
@@
 		(in_pos_files yes)
 		(dnp no)
-		(property "Reference" "R33"
+		(property "Reference" "R35"
 			(at 95.504 85.09 0)
 			(show_name no)
@@
 			(project "Main_Board"
 				(path "/7481738f-7c20-40bb-99b0-6ccd4168db33/f339aa79-d1b1-4b60-b951-815db04e9281/9134e59b-c18f-4136-baaa-a4c593015be7"
-					(reference "R33")
+					(reference "R35")
 					(unit 1)
 				)
@@
 		(in_pos_files yes)
 		(dnp no)
-		(property "Reference" "#PWR087"
+		(property "Reference" "#PWR091"
 			(at 110.49 95.25 0)
 			(hide yes)
@@
 			(project "Main_Board"
 				(path "/7481738f-7c20-40bb-99b0-6ccd4168db33/f339aa79-d1b1-4b60-b951-815db04e9281/9134e59b-c18f-4136-baaa-a4c593015be7"
-					(reference "#PWR087")
-					(unit 1)
-				)
+					(reference "#PWR091")
+					(unit 1)
+				)

Commit message: Standardise resistor value mark for BOM + pyro footprints
Parts:
- R35, R36: value 10K -> 10k
Changed lines of the file:
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@@
 			)
 		)
-		(property "Value" "10K"
+		(property "Value" "10k"
 			(at 129.794 112.776 0)
 			(show_name no)
@@
 			)
 		)
-		(property "Value" "10K"
+		(property "Value" "10k"
 			(at 95.504 87.376 0)
 			(show_name no)

Commit message: fix after review -?D7/D8 clamp to 3v3 MB not for 3v3 and other fix
Parts:
- U7: value THVD1450DR -> TLV61070A
Changed lines of the file:
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@@
 			)
 		)
-		(property "Value" "THVD1450DR"
+		(property "Value" "TLV61070A"
 			(at 151.13 118.11 0)
 			(show_name no)

Commit message: ALED Level shifter, fix RS485 transciever IC naming
Parts:
- U7: value TLV61070A -> THVD1450DRBR
Changed lines of the file:
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@@
 			)
 		)
-		(property "Value" "TLV61070A"
+		(property "Value" "THVD1450DRBR"
 			(at 151.13 118.11 0)
 			(show_name no)
