File: Main_Board/Boost.kicad_sch (KiCad schematic)
At the start: 13 parts, among them U5 TLV61070ADBV

Commit message: Cap note
Other:
- note added: "C23-C25 = GRM188R61A106MAAL"
Changed lines of the file:
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@@
 	(text "Inductor: Murata DFE322520FD-2R2M=P2"
 		(exclude_from_sim no)
-		(at 134.112 74.93 0)
+		(at 134.366 75.184 0)
 		(effects
 			(font
+				(size 1.27 1.27)
+			)
+		)
+	)
+	(text "C23-C25 = GRM188R61A106MAAL"
+		(exclude_from_sim no)
+		(at 182.626 92.202 0)
+		(effects
+			(font
